Commit message: rename RealSense D435i frames camera_* -> realsense_*

File: xarm_description/urdf/camera/realsense.gazebo.xacro (robot description, xacro)
@@ -2,5 +2,5 @@
 <robot xmlns:xacro="http://ros.org/wiki/xacro">
   <xacro:macro name="realsense_gazebo" params="prefix:=''">
-    <gazebo reference="${prefix}camera_depth_frame">
+    <gazebo reference="${prefix}realsense_depth_frame">
       <sensor name="${prefix}cameradepth" type="depth">
         <camera name="${prefix}camera">
@@ -25,5 +25,5 @@
       </sensor>
     </gazebo>
-    <gazebo reference="${prefix}camera_color_frame">
+    <gazebo reference="${prefix}realsense_color_frame">
       <sensor name="${prefix}cameracolor" type="camera">
         <camera name="${prefix}camera">
@@ -49,5 +49,5 @@
       </sensor>
     </gazebo>
-    <gazebo reference="${prefix}camera_left_ir_frame">
+    <gazebo reference="${prefix}realsense_left_ir_frame">
       <sensor name="${prefix}cameraired1" type="camera">
         <camera name="${prefix}camera">
@@ -73,5 +73,5 @@
       </sensor>
     </gazebo>
-    <gazebo reference="${prefix}camera_right_ir_frame">
+    <gazebo reference="${prefix}realsense_right_ir_frame">
       <sensor name="${prefix}cameraired2" type="camera">
         <camera name="${prefix}camera">
@@ -111,8 +111,8 @@
         <infrared2TopicName>${prefix}infra2/image_raw</infrared2TopicName>
         <infrared2CameraInfoTopicName>${prefix}infra2/camera_info</infrared2CameraInfoTopicName>
-        <colorOpticalframeName>${prefix}camera_color_optical_frame</colorOpticalframeName>
-        <depthOpticalframeName>${prefix}camera_depth_optical_frame</depthOpticalframeName>
-        <infrared1OpticalframeName>${prefix}camera_left_ir_optical_frame</infrared1OpticalframeName>
-        <infrared2OpticalframeName>${prefix}camera_right_ir_optical_frame</infrared2OpticalframeName>
+        <colorOpticalframeName>${prefix}realsense_color_optical_frame</colorOpticalframeName>
+        <depthOpticalframeName>${prefix}realsense_depth_optical_frame</depthOpticalframeName>
+        <infrared1OpticalframeName>${prefix}realsense_left_ir_optical_frame</infrared1OpticalframeName>
+        <infrared2OpticalframeName>${prefix}realsense_right_ir_optical_frame</infrared2OpticalframeName>
         <rangeMinDepth>0.3</rangeMinDepth>
         <rangeMaxDepth>3.0</rangeMaxDepth>
@@ -124,5 +124,5 @@
   </xacro:macro>
   <xacro:macro name="realsense_ignition" params="prefix:=''">
-    <gazebo reference="${prefix}camera_depth_frame">
+    <gazebo reference="${prefix}realsense_depth_frame">
       <sensor name="${prefix}cameradepth" type="rgbd_camera">
         <camera name="${prefix}camera">
@@ -156,8 +156,8 @@
       </sensor>
     </gazebo>
-    <gazebo reference="${prefix}camera_color_frame">
+    <gazebo reference="${prefix}realsense_color_frame">
       <sensor name="${prefix}cameracolor" type="camera">
-        <!-- <ignition_frame_id>${prefix}camera_color_frame</ignition_frame_id>
-        <optical_frame_id>${prefix}camera_color_frame</optical_frame_id> -->
+        <!-- <ignition_frame_id>${prefix}realsense_color_frame</ignition_frame_id>
+        <optical_frame_id>${prefix}realsense_color_frame</optical_frame_id> -->
         <camera name="${prefix}camera">
           <horizontal_fov>1.57</horizontal_fov>
@@ -185,5 +185,5 @@
       </sensor>
     </gazebo>
-    <gazebo reference="${prefix}camera_left_ir_frame">
+    <gazebo reference="${prefix}realsense_left_ir_frame">
       <sensor name="${prefix}cameraired1" type="camera">
         <camera name="${prefix}camera">
@@ -211,5 +211,5 @@
       </sensor>
     </gazebo>
-    <gazebo reference="${prefix}camera_right_ir_frame">
+    <gazebo reference="${prefix}realsense_right_ir_frame">
       <sensor name="${prefix}cameraired2" type="camera">
         <camera name="${prefix}camera">
@@ -246,5 +246,5 @@
   </xacro:macro>
   <xacro:macro name="realsense_gz" params="prefix:=''">
-    <gazebo reference="${prefix}camera_depth_frame">
+    <gazebo reference="${prefix}realsense_depth_frame">
       <sensor name="${prefix}cameradepth" type="rgbd_camera">
         <camera name="${prefix}camera">
@@ -278,8 +278,8 @@
       </sensor>
     </gazebo>
-    <gazebo reference="${prefix}camera_color_frame">
+    <gazebo reference="${prefix}realsense_color_frame">
       <sensor name="${prefix}cameracolor" type="camera">
-        <!-- <ignition_frame_id>${prefix}camera_color_frame</ignition_frame_id>
-        <optical_frame_id>${prefix}camera_color_frame</optical_frame_id> -->
+        <!-- <ignition_frame_id>${prefix}realsense_color_frame</ignition_frame_id>
+        <optical_frame_id>${prefix}realsense_color_frame</optical_frame_id> -->
         <camera name="${prefix}camera">
           <horizontal_fov>1.57</horizontal_fov>
@@ -307,5 +307,5 @@
       </sensor>
     </gazebo>
-    <gazebo reference="${prefix}camera_left_ir_frame">
+    <gazebo reference="${prefix}realsense_left_ir_frame">
       <sensor name="${prefix}cameraired1" type="camera">
         <camera name="${prefix}camera">
@@ -333,5 +333,5 @@
       </sensor>
     </gazebo>
-    <gazebo reference="${prefix}camera_right_ir_frame">
+    <gazebo reference="${prefix}realsense_right_ir_frame">
       <sensor name="${prefix}cameraired2" type="camera">
         <camera name="${prefix}camera">

File: xarm_description/urdf/camera/realsense_d435i.urdf.xacro (robot description, xacro)
@@ -16,56 +16,56 @@
     </link>
     <xacro:if value="${add_d435i_links}">
-      <link name="${prefix}camera_link"></link>
-      <link name="${prefix}camera_depth_frame"></link>
-      <link name="${prefix}camera_depth_optical_frame"></link>
-      <link name="${prefix}camera_color_frame"></link>
-      <link name="${prefix}camera_color_optical_frame"></link>
-      <link name="${prefix}camera_left_ir_frame"></link>
-      <link name="${prefix}camera_left_ir_optical_frame"></link>
-      <link name="${prefix}camera_right_ir_frame"></link>
-      <link name="${prefix}camera_right_ir_optical_frame"></link>
-      <joint name="${prefix}camera_link_joint" type="fixed">
+      <link name="${prefix}realsense_link"></link>
+      <link name="${prefix}realsense_depth_frame"></link>
+      <link name="${prefix}realsense_depth_optical_frame"></link>
+      <link name="${prefix}realsense_color_frame"></link>
+      <link name="${prefix}realsense_color_optical_frame"></link>
+      <link name="${prefix}realsense_left_ir_frame"></link>
+      <link name="${prefix}realsense_left_ir_optical_frame"></link>
+      <link name="${prefix}realsense_right_ir_frame"></link>
+      <link name="${prefix}realsense_right_ir_optical_frame"></link>
+      <joint name="${prefix}realsense_link_joint" type="fixed">
         <parent link="${prefix}link_eef" />
-        <child link="${prefix}camera_link" />
+        <child link="${prefix}realsense_link" />
         <origin xyz="0.06746 -0.0175 0.0237" rpy="${M_PI} ${-M_PI/2} 0" />
       </joint>
-      <joint name="${prefix}camera_depth_joint" type="fixed">
-        <parent link="${prefix}camera_link" />
-        <child link="${prefix}camera_depth_frame" />
+      <joint name="${prefix}realsense_depth_joint" type="fixed">
+        <parent link="${prefix}realsense_link" />
+        <child link="${prefix}realsense_depth_frame" />
         <origin xyz="0 0 0" rpy="0 0 0" />
       </joint>
-      <joint name="${prefix}camera_depth_optical_joint" type="fixed">
-        <parent link="${prefix}camera_depth_frame" />
-        <child link="${prefix}camera_depth_optical_frame" />
+      <joint name="${prefix}realsense_depth_optical_joint" type="fixed">
+        <parent link="${prefix}realsense_depth_frame" />
+        <child link="${prefix}realsense_depth_optical_frame" />
         <origin xyz="0 0 0" rpy="${-M_PI/2} 0 ${-M_PI/2}" />
       </joint>
-      <joint name="${prefix}camera_color_joint" type="fixed">
-        <parent link="${prefix}camera_link" />
-        <child link="${prefix}camera_color_frame" />
+      <joint name="${prefix}realsense_color_joint" type="fixed">
+        <parent link="${prefix}realsense_link" />
+        <child link="${prefix}realsense_color_frame" />
         <origin xyz="0 0.015 0" rpy="0 0 0" />
       </joint>
-      <joint name="${prefix}camera_color_optical_joint" type="fixed">
-        <parent link="${prefix}camera_color_frame" />
-        <child link="${prefix}camera_color_optical_frame" />
+      <joint name="${prefix}realsense_color_optical_joint" type="fixed">
+        <parent link="${prefix}realsense_color_frame" />
+        <child link="${prefix}realsense_color_optical_frame" />
         <origin xyz="0 0 0" rpy="${-M_PI/2} 0 ${-M_PI/2}" />
       </joint>
-      <joint name="${prefix}camera_left_ir_joint" type="fixed">
-        <parent link="${prefix}camera_link" />
-        <child link="${prefix}camera_left_ir_frame" />
+      <joint name="${prefix}realsense_left_ir_joint" type="fixed">
+        <parent link="${prefix}realsense_link" />
+        <child link="${prefix}realsense_left_ir_frame" />
         <origin xyz="0 0 0" rpy="0 0 0" />
       </joint>
-      <joint name="${prefix}camera_left_ir_optical_joint" type="fixed">
-        <parent link="${prefix}camera_left_ir_frame" />
-        <child link="${prefix}camera_left_ir_optical_frame" />
+      <joint name="${prefix}realsense_left_ir_optical_joint" type="fixed">
+        <parent link="${prefix}realsense_left_ir_frame" />
+        <child link="${prefix}realsense_left_ir_optical_frame" />
         <origin xyz="0 0 0" rpy="${-M_PI/2} 0 ${-M_PI/2}" />
       </joint>
-      <joint name="${prefix}camera_right_ir_joint" type="fixed">
-        <parent link="${prefix}camera_link" />
-        <child link="${prefix}camera_right_ir_frame" />
+      <joint name="${prefix}realsense_right_ir_joint" type="fixed">
+        <parent link="${prefix}realsense_link" />
+        <child link="${prefix}realsense_right_ir_frame" />
         <origin xyz="0 -0.050 0" rpy="0 0 0" />
       </joint>
-      <joint name="${prefix}camera_right_ir_optical_joint" type="fixed">
-        <parent link="${prefix}camera_right_ir_frame" />
-        <child link="${prefix}camera_right_ir_optical_frame" />
+      <joint name="${prefix}realsense_right_ir_optical_joint" type="fixed">
+        <parent link="${prefix}realsense_right_ir_frame" />
+        <child link="${prefix}realsense_right_ir_optical_frame" />
         <origin xyz="0 0 0" rpy="${-M_PI/2} 0 ${-M_PI/2}" />
       </joint>
