Commit message: xarm6 srdf: add saved arm poses

File: xarm_moveit_config/srdf/_xarm6_macro.srdf.xacro (robot description, xacro)
@@ -54,4 +54,60 @@
       <joint name="${prefix}joint5" value="-1.5708" />
       <joint name="${prefix}joint6" value="0" />
+    </group_state>
+    <group_state name="test" group="${prefix}xarm6">
+      <joint name="${prefix}joint1" value="-1.5708" />
+      <joint name="${prefix}joint2" value="0" />
+      <joint name="${prefix}joint3" value="0" />
+      <joint name="${prefix}joint4" value="0" />
+      <joint name="${prefix}joint5" value="0" />
+      <joint name="${prefix}joint6" value="0" />
+    </group_state>
+    <group_state name="here" group="${prefix}xarm6">
+      <joint name="${prefix}joint1" value="-1.707347498391325" />
+      <joint name="${prefix}joint2" value="0.3024435365458249" />
+      <joint name="${prefix}joint3" value="-0.66842466580390303" />
+      <joint name="${prefix}joint4" value="3.0717990939032909" />
+      <joint name="${prefix}joint5" value="2.4399011008507574" />
+      <joint name="${prefix}joint6" value="1.6463648359368004" />
+    </group_state>
+    <group_state name="test_pr" group="${prefix}xarm6">
+      <joint name="${prefix}joint1" value="0" />
+      <joint name="${prefix}joint2" value="0" />
+      <joint name="${prefix}joint3" value="0" />
+      <joint name="${prefix}joint4" value="0" />
+      <joint name="${prefix}joint5" value="0" />
+      <joint name="${prefix}joint6" value="0" />
+    </group_state>
+    <group_state name="desired" group="${prefix}xarm6">
+      <joint name="${prefix}joint1" value="0" />
+      <joint name="${prefix}joint2" value="0" />
+      <joint name="${prefix}joint3" value="0" />
+      <joint name="${prefix}joint4" value="0" />
+      <joint name="${prefix}joint5" value="0" />
+      <joint name="${prefix}joint6" value="0" />
+    </group_state>
+    <group_state name="pose1" group="${prefix}xarm6">
+      <joint name="${prefix}joint1" value="0" />
+      <joint name="${prefix}joint2" value="0" />
+      <joint name="${prefix}joint3" value="0" />
+      <joint name="${prefix}joint4" value="0" />
+      <joint name="${prefix}joint5" value="0" />
+      <joint name="${prefix}joint6" value="0" />
+    </group_state>
+    <group_state name="Drop" group="${prefix}xarm6">
+      <joint name="${prefix}joint1" value="-1.441153883934021" />
+      <joint name="${prefix}joint2" value="1.1510416269302368" />
+      <joint name="${prefix}joint3" value="-2.1076436042785645" />
+      <joint name="${prefix}joint4" value="0.2316330224275589" />
+      <joint name="${prefix}joint5" value="-0.62697052955627441" />
+      <joint name="${prefix}joint6" value="-0.18862402439117432" />
+    </group_state>
+    <group_state name="DropBottle" group="${prefix}xarm6">
+      <joint name="${prefix}joint1" value="0.040918938815593719" />
+      <joint name="${prefix}joint2" value="0.86983036994934082" />
+      <joint name="${prefix}joint3" value="-1.8259931802749634" />
+      <joint name="${prefix}joint4" value="-0.02351592481136322" />
+      <joint name="${prefix}joint5" value="-0.64023375511169434" />
+      <joint name="${prefix}joint6" value="2.3009712094790302e-05" />
     </group_state>
     <!-- gripper -->
